Commit message: work in ROS2 humble

File: launch/ego_racecar_f1fifth.xacro (robot description, xacro)
@@ -2,14 +2,13 @@
 <!-- A simple model of the racecar for rviz -->
 <robot xmlns:xacro="http://www.ros.org/wiki/xacro" name="racecar">
-  <xacro:property name="wheelbase" value="0.32" />
-  <xacro:property name="width" value="0.28" />
-  <xacro:property name="length" value="0.51" />
-  <xacro:property name="height" value="0.1" />
-  <xacro:property name="ground_offset" value="0.04" />
-  <xacro:property name="wheel_radius" value="0.0508" />
-  <xacro:property name="wheel_length" value="0.0381" />
-  <xacro:property name="laser_distance_from_base_link" value="0.275" />
-  <xacro:property name="laser_height" value="0.05" />
-  <xacro:property name="laser_radius" value="0.026" />
+  <xacro:property name="wheelbase" value="0.532" />
+  <xacro:property name="width" value="0.54" />
+  <xacro:property name="height" value="0.3" />
+  <xacro:property name="ground_offset" value="0.107" />
+  <xacro:property name="wheel_radius" value="0.145" />
+  <xacro:property name="wheel_length" value="0.110" />
+  <xacro:property name="laser_distance_from_base_link" value="0.45" />
+  <xacro:property name="laser_height" value="0.09" />
+  <xacro:property name="laser_radius" value="0.054" />
   <xacro:property name="car_name" value="ego_racecar" />
   <material name="black">
@@ -21,7 +20,7 @@
   <link name="${car_name}/base_link">
     <visual>
-      <origin xyz="0 0 ${ground_offset+height/2}"/>
+      <origin xyz="${wheelbase/2} 0 ${ground_offset+height/2}"/>
       <geometry>
-        <box size="${length} ${width} ${height}"/>
+        <box size="${wheelbase} ${width} ${height}"/>
       </geometry>
       <material name="blue"/>
@@ -31,5 +30,5 @@
     <parent link="${car_name}/base_link"/>
     <child link="${car_name}/laser_model"/>
-    <origin xyz="${laser_distance_from_base_link-wheelbase/2} 0 ${ground_offset+height+(laser_height/2)}"/>
+    <origin xyz="${laser_distance_from_base_link} 0 ${ground_offset+height+(laser_height/2)}"/>
   </joint>
   <link name="${car_name}/laser_model">
@@ -44,5 +43,5 @@
     <parent link="${car_name}/base_link"/>
     <child link="${car_name}/back_left_wheel"/>
-    <origin xyz="${-wheelbase/2} ${(wheel_length+width)/2} ${wheel_radius}"/>
+    <origin xyz="0 ${(wheel_length+width)/2} ${wheel_radius}"/>
   </joint>
   <link name="${car_name}/back_left_wheel">
@@ -58,5 +57,5 @@
     <parent link="${car_name}/base_link"/>
     <child link="${car_name}/back_right_wheel"/>
-    <origin xyz="${-wheelbase/2} ${-(wheel_length+width)/2} ${wheel_radius}"/>
+    <origin xyz="0 ${-(wheel_length+width)/2} ${wheel_radius}"/>
   </joint>
   <link name="${car_name}/back_right_wheel">
@@ -72,5 +71,5 @@
     <parent link="${car_name}/base_link"/>
     <child link="${car_name}/front_left_hinge"/>
-    <origin xyz="${wheelbase/2} ${(wheel_length+width)/2} ${wheel_radius}"/>
+    <origin xyz="${wheelbase} ${(wheel_length+width)/2} ${wheel_radius}"/>
   </joint>
   <link name="${car_name}/front_left_hinge"/>
@@ -91,5 +90,5 @@
     <parent link="${car_name}/base_link"/>
     <child link="${car_name}/front_right_hinge"/>
-    <origin xyz="${wheelbase/2} ${-(wheel_length+width)/2} ${wheel_radius}"/>
+    <origin xyz="${wheelbase} ${-(wheel_length+width)/2} ${wheel_radius}"/>
   </joint>
   <link name="${car_name}/front_right_hinge"/>

File: launch/ego_racecar_fullscale.xacro (robot description, xacro)
@@ -2,14 +2,13 @@
 <!-- A simple model of the racecar for rviz -->
 <robot xmlns:xacro="http://www.ros.org/wiki/xacro" name="racecar">
-  <xacro:property name="wheelbase" value="0.32" />
-  <xacro:property name="width" value="0.28" />
-  <xacro:property name="length" value="0.51" />
-  <xacro:property name="height" value="0.1" />
-  <xacro:property name="ground_offset" value="0.04" />
-  <xacro:property name="wheel_radius" value="0.0508" />
-  <xacro:property name="wheel_length" value="0.0381" />
-  <xacro:property name="laser_distance_from_base_link" value="0.275" />
-  <xacro:property name="laser_height" value="0.05" />
-  <xacro:property name="laser_radius" value="0.026" />
+  <xacro:property name="wheelbase" value="2.39268" /> <!-- TODO: change to full scale params -->
+  <xacro:property name="width" value="1.64" />
+  <xacro:property name="height" value="1.32" />
+  <xacro:property name="ground_offset" value="0.14986" />
+  <xacro:property name="wheel_radius" value="0.381" />
+  <xacro:property name="wheel_length" value="0.1397" />
+  <xacro:property name="laser_distance_from_base_link" value="2.0" />
+  <xacro:property name="laser_height" value="0.09" />
+  <xacro:property name="laser_radius" value="0.054" />
   <xacro:property name="car_name" value="ego_racecar" />
   <material name="black">
@@ -21,7 +20,7 @@
   <link name="${car_name}/base_link">
     <visual>
-      <origin xyz="0 0 ${ground_offset+height/2}"/>
+      <origin xyz="${wheelbase/2} 0 ${ground_offset+height/2}"/>
       <geometry>
-        <box size="${length} ${width} ${height}"/>
+        <box size="${wheelbase} ${width} ${height}"/>
       </geometry>
       <material name="blue"/>
@@ -31,5 +30,5 @@
     <parent link="${car_name}/base_link"/>
     <child link="${car_name}/laser_model"/>
-    <origin xyz="${laser_distance_from_base_link-wheelbase/2} 0 ${ground_offset+height+(laser_height/2)}"/>
+    <origin xyz="${laser_distance_from_base_link} 0 ${ground_offset+height+(laser_height/2)}"/>
   </joint>
   <link name="${car_name}/laser_model">
@@ -44,5 +43,5 @@
     <parent link="${car_name}/base_link"/>
     <child link="${car_name}/back_left_wheel"/>
-    <origin xyz="${-wheelbase/2} ${(wheel_length+width)/2} ${wheel_radius}"/>
+    <origin xyz="0 ${(wheel_length+width)/2} ${wheel_radius}"/>
   </joint>
   <link name="${car_name}/back_left_wheel">
@@ -58,5 +57,5 @@
     <parent link="${car_name}/base_link"/>
     <child link="${car_name}/back_right_wheel"/>
-    <origin xyz="${-wheelbase/2} ${-(wheel_length+width)/2} ${wheel_radius}"/>
+    <origin xyz="0 ${-(wheel_length+width)/2} ${wheel_radius}"/>
   </joint>
   <link name="${car_name}/back_right_wheel">
@@ -72,5 +71,5 @@
     <parent link="${car_name}/base_link"/>
     <child link="${car_name}/front_left_hinge"/>
-    <origin xyz="${wheelbase/2} ${(wheel_length+width)/2} ${wheel_radius}"/>
+    <origin xyz="${wheelbase} ${(wheel_length+width)/2} ${wheel_radius}"/>
   </joint>
   <link name="${car_name}/front_left_hinge"/>
@@ -91,5 +90,5 @@
     <parent link="${car_name}/base_link"/>
     <child link="${car_name}/front_right_hinge"/>
-    <origin xyz="${wheelbase/2} ${-(wheel_length+width)/2} ${wheel_radius}"/>
+    <origin xyz="${wheelbase} ${-(wheel_length+width)/2} ${wheel_radius}"/>
   </joint>
   <link name="${car_name}/front_right_hinge"/>

File: launch/opp_racecar.xacro (robot description, xacro)
@@ -2,6 +2,7 @@
 <!-- A simple model of the racecar for rviz -->
 <robot xmlns:xacro="http://www.ros.org/wiki/xacro" name="racecar">
-  <xacro:property name="wheelbase" value="0.3302" />
-  <xacro:property name="width" value="0.2032" />
+  <xacro:property name="wheelbase" value="0.32" />
+  <xacro:property name="width" value="0.28" />
+  <xacro:property name="length" value="0.51" />
   <xacro:property name="height" value="0.1" />
   <xacro:property name="ground_offset" value="0.04" />
@@ -20,9 +21,9 @@
   <link name="${car_name}/base_link">
     <visual>
-      <origin xyz="${wheelbase/2} 0 ${ground_offset+height/2}"/>
+      <origin xyz="0 0 ${ground_offset+height/2}"/>
       <geometry>
-        <box size="${wheelbase} ${width} ${height}"/>
+        <box size="${length} ${width} ${height}"/>
       </geometry>
-      <material name="red"/>
+      <material name="blue"/>
     </visual>
   </link>
@@ -30,5 +31,5 @@
     <parent link="${car_name}/base_link"/>
     <child link="${car_name}/laser_model"/>
-    <origin xyz="${laser_distance_from_base_link} 0 ${ground_offset+height+(laser_height/2)}"/>
+    <origin xyz="${laser_distance_from_base_link-wheelbase/2} 0 ${ground_offset+height+(laser_height/2)}"/>
   </joint>
   <link name="${car_name}/laser_model">
@@ -43,5 +44,5 @@
     <parent link="${car_name}/base_link"/>
     <child link="${car_name}/back_left_wheel"/>
-    <origin xyz="0 ${(wheel_length+width)/2} ${wheel_radius}"/>
+    <origin xyz="${-wheelbase/2} ${(wheel_length+width)/2} ${wheel_radius}"/>
   </joint>
   <link name="${car_name}/back_left_wheel">
@@ -57,5 +58,5 @@
     <parent link="${car_name}/base_link"/>
     <child link="${car_name}/back_right_wheel"/>
-    <origin xyz="0 ${-(wheel_length+width)/2} ${wheel_radius}"/>
+    <origin xyz="${-wheelbase/2} ${-(wheel_length+width)/2} ${wheel_radius}"/>
   </joint>
   <link name="${car_name}/back_right_wheel">
@@ -71,5 +72,5 @@
     <parent link="${car_name}/base_link"/>
     <child link="${car_name}/front_left_hinge"/>
-    <origin xyz="${wheelbase} ${(wheel_length+width)/2} ${wheel_radius}"/>
+    <origin xyz="${wheelbase/2} ${(wheel_length+width)/2} ${wheel_radius}"/>
   </joint>
   <link name="${car_name}/front_left_hinge"/>
@@ -90,5 +91,5 @@
     <parent link="${car_name}/base_link"/>
     <child link="${car_name}/front_right_hinge"/>
-    <origin xyz="${wheelbase} ${-(wheel_length+width)/2} ${wheel_radius}"/>
+    <origin xyz="${wheelbase/2} ${-(wheel_length+width)/2} ${wheel_radius}"/>
   </joint>
   <link name="${car_name}/front_right_hinge"/>
